File: KBD8X-MK2-aek.kicad_pcb (KiCad board)
At the start: 2 copper layers, 343.7 x 118.3 mm, 205 parts, among them J1 AVR-ISP-6, Q1 DSS60601MZ4-13, SW1 SW_Push, U1 ATmega32U4-MU, U2 PRTR5V0U2X, Y1 16MHz

Commit message: route some bottom row stuff + add pads ratnest
Parts:
- moved D84 26.1 mm to (60.5, 138.9)
- moved D91 5.00 mm to (249.0, 138.9)
- moved D85 3.55 mm to (86.9, 138.9)
Connections:
- MX_LALT2 pad 2: (no net) -> COL1
- MX_LGUI2 pad 1: (no net) -> COL0
- MX_LGUI2 pad 2: (no net) -> Net-(D85-Pad2)
- MX_RALT2 pad 1: (no net) -> Net-(D91-Pad2)
- MX_RGUI2 pad 1: (no net) -> COL6
Routing:
- net ROW10: track 304.3 -> 332.0 mm
- net Net-(D84-Pad2): track 34.1 -> 6.56 mm
- net COL1: track 270.0 -> 282.0 mm
- net COL0: track 201.3 -> 206.0 mm
- net ROW11: track 318.6 -> 314.6 mm
- net Net-(D85-Pad2): track 5.43 -> 8.99 mm
- net COL6: track 374.3 -> 376.7 mm
- net Net-(D52-Pad2): track 20.2 -> 22.4 mm
- net COL3: track 437.4 -> 435.6 mm, vias 1 -> 0
- net Net-(D91-Pad2): track 12.4 -> 11.7 mm

Commit message: south facing standard, north facing aek bottom row, south facing alps caps lock
Parts:
- added MX_LCTRL1: MX-ALPS-1.5U, MX_Alps_Hybrid:MX-1.25U-NoLED, F.Cu at (97.6, 139.7)
- added MX_LCTRL1: MX-ALPS-1.5U, MX_Alps_Hybrid:MX-1.25U-NoLED, F.Cu at (50.0, 139.7)
- added MX_LCTRL1: MX-ALPS-1.5U, MX_Alps_Hybrid:MX-1.25U-NoLED, F.Cu at (73.8, 139.7)
- added MX_SP2: MX-7U, MX_Alps_Hybrid:MX-6.25U-NoLED, F.Cu at (169.1, 139.7)
- moved D86 23.8 mm to (113.5, 138.9)
- moved D87 10.2 mm to (160.9, 139.0)
- moved G*** 4.00 mm to (140.7, 137.8)
- turned MX_CLOCK2 to 180 degrees
Connections:
- MX_CLOCK2 pad : COL0 -> Net-(D52-Pad2)
- MX_LALT2 pad 1: (no net) -> Net-(D86-Pad2)
Routing:
- net COL0: track 206.0 -> 236.3 mm
- net ROW10: track 332.0 -> 348.6 mm, vias 2 -> 4
- net COL3: track 435.6 -> 450.4 mm
- net Net-(D85-Pad2): track 8.99 -> 23.7 mm
- net Net-(D87-Pad2): track 14.2 -> 28.5 mm
- net Net-(D86-Pad2): track 14.7 -> 28.2 mm
- net Net-(D84-Pad2): track 6.56 -> 18.6 mm
- net COL1: track 282.0 -> 293.4 mm
- net Net-(D52-Pad2): track 22.4 -> 29.6 mm
- net ROW11: track 314.6 -> 321.0 mm
Other:
- board text added: "Rogue x ai03"
