File: matrix.kicad_sch (KiCad schematic)
At the start: 285 parts, among them SW2 SW_SPDT, SW3 SW_SPDT

Commit message: move f1 + many split layout to complex version, add more board ocmponents
Parts:
- removed R1, R10, R100, R101, R108, R11, R111, R112, R113, R12, R13, R14, R16, R17, R18, R19, R2, R20, R21, R22, R23, R24, R25, R26, R27, R28, R29, R3, R30, R31, R32, R33, R35, R36, R37, R38, R39, R4, R40, R41, R42, R43, R44, R45, R46, R47, R48, R5, R53, R54, R55, R56, R57, R58, R59, R6, R60, R61, R62, R63, R65, R66, R67, R68, R69, R7, R70, R71, R72, R73, R74, R75, R76, R77, R78, R8, R81, R82, R84, R85, R86, R87, R9, R90, R91, R95, R96, R97, R99: 1k, locallib:R_0603, symbol Device:R_Small
- removed SW2: SW_SPDT, Buttons_Switches_SMD:SW_SPDT_PCM12, symbol Switch:SW_SPDT
- added MX_CLOCK3: MX-1.5U, MX_Alps_Hybrid:MXOnly-1.25U-FLIPPED, symbol MX_Alps_Hybrids:MX-1.25U
- added MX_LALT3: MX-1.5U, MX_Alps_Hybrid:MXOnly-1U-FLIPPED, symbol MX_Alps_Hybrid:MX-NoLED
- added MX_LCTRL3: MX-1.5U, MX_Alps_Hybrid:MXOnly-1.5U-FLIPPED, symbol MX_Alps_Hybrid:MX-NoLED
- added MX_LGUI3: MX-1.25U, MX_Alps_Hybrid:MXOnly-1U-FLIPPED, symbol MX_Alps_Hybrid:MX-NoLED
- added MX_RALT3, MX_RCTRL?: MX-1.5U, MX_Alps_Hybrid:MXOnly-1.5U, symbol MX_Alps_Hybrid:MX-NoLED
- added MX_RGUI?: MX-1U, MX_Alps_Hybrid:MXOnly-1U, symbol MX_Alps_Hybrid:MX-NoLED
- added MX_SP3: MX-6.5U, MX_Alps_Hybrid:MXOnly-7U-ReversedStabilizers, symbol MX_Alps_Hybrid:MX-NoLED
- MX_#0_1, MX_#1, MX_#2, MX_#3, MX_#4, MX_#5, MX_#6, MX_#7, MX_#8, MX_#9, MX_'1, MX_,1, MX_-1, MX_.1, MX_/1, MX_;1, MX_=1, MX_A1, MX_B1, MX_BACK2, MX_BACK3, MX_C1, MX_D1, MX_DEL1, MX_DN1, MX_E1, MX_END1, MX_ESC1, MX_F1, MX_FN1, MX_FN10, MX_FN11, MX_FN12, MX_FN2, MX_FN3, MX_FN4, MX_FN5, MX_FN6, MX_FN7, MX_FN8, MX_FN9, MX_G1, MX_H1, MX_HOME1, MX_I1, MX_INS1, MX_J1, MX_K1, MX_L1, MX_LCTRL1, MX_LFT1, MX_LSHIFT3, MX_M1, MX_N1, MX_O1, MX_P1, MX_PAUSE1, MX_PGDN1, MX_PGUP1, MX_PRINT1, MX_Q1, MX_R1, MX_RCTRL1, MX_RMENU1, MX_RSHIFT1, MX_RSHIFT2, MX_RSHIFT3, MX_RT1, MX_S1, MX_SLOCK1, MX_T1, MX_U1, MX_UP1, MX_V1, MX_W1, MX_X1, MX_Y1, MX_Z1, MX_[1, MX_\2, MX_]1, MX_`1: symbol MX_Alps_Hybrids:MX-1U -> MX_Alps_Hybrid:MX-NoLED
- MX_BACK1: symbol MX_Alps_Hybrids:MX-2U -> MX_Alps_Hybrid:MX-NoLED
- MX_LALT1, MX_LGUI1, MX_RALT1, MX_RGUI1: symbol MX_Alps_Hybrids:MX-1.25U -> MX_Alps_Hybrid:MX-NoLED
- MX_LALT2, MX_LCTRL2, MX_LGUI2, MX_RALT2, MX_RCTRL2, MX_RGUI2, MX_TAB1, MX_\1: symbol MX_Alps_Hybrids:MX-1.5U -> MX_Alps_Hybrid:MX-NoLED
- MX_LSHIFT1, MX_LSHIFT2, MX_RETURN1, MX_RETURN2: symbol MX_Alps_Hybrids:MX-2.25U -> MX_Alps_Hybrid:MX-NoLED
- MX_SP1: symbol MX_Alps_Hybrids:MX-6.25U -> MX_Alps_Hybrid:MX-NoLED
- MX_SP2: symbol MX_Alps_Hybrids:MX-7U -> MX_Alps_Hybrid:MX-NoLED
Connections:
- net +5V: now also MX_CLOCK3.3 (LED); no longer MX_#0_1.3 (LED), MX_#1.3 (LED), MX_#2.3 (LED), MX_#3.3 (LED), MX_#4.3 (LED), MX_#5.3 (LED), MX_#6.3 (LED), MX_#7.3 (LED), MX_#8.3 (LED), MX_#9.3 (LED), MX_'1.3 (LED), MX_,1.3 (LED), MX_-1.3 (LED), MX_.1.3 (LED), MX_/1.3 (LED), MX_;1.3 (LED), MX_=1.3 (LED), MX_A1.3 (LED), MX_B1.3 (LED), MX_BACK1.3 (LED), MX_BACK2.3 (LED), MX_BACK3.3 (LED), MX_C1.3 (LED), MX_D1.3 (LED), MX_DEL1.3 (LED), MX_DN1.3 (LED), MX_E1.3 (LED), MX_END1.3 (LED), MX_ESC1.3 (LED), MX_F1.3 (LED), MX_FN1.3 (LED), MX_FN10.3 (LED), MX_FN11.3 (LED), MX_FN12.3 (LED), MX_FN2.3 (LED), MX_FN3.3 (LED), MX_FN4.3 (LED), MX_FN5.3 (LED), MX_FN6.3 (LED), MX_FN7.3 (LED), MX_FN8.3 (LED), MX_FN9.3 (LED), MX_G1.3 (LED), MX_H1.3 (LED), MX_HOME1.3 (LED), MX_I1.3 (LED), MX_INS1.3 (LED), MX_J1.3 (LED), MX_K1.3 (LED), MX_L1.3 (LED), MX_LALT1.3 (LED), MX_LALT2.3 (LED), MX_LCTRL1.3 (LED), MX_LCTRL2.3 (LED), MX_LFT1.3 (LED), MX_LGUI1.3 (LED), MX_LGUI2.3 (LED), MX_LSHIFT1.3 (LED), MX_LSHIFT2.3 (LED), MX_LSHIFT3.3 (LED), MX_M1.3 (LED), MX_N1.3 (LED), MX_O1.3 (LED), MX_P1.3 (LED), MX_PAUSE1.3 (LED), MX_PGDN1.3 (LED), MX_PGUP1.3 (LED), MX_PRINT1.3 (LED), MX_Q1.3 (LED), MX_R1.3 (LED), MX_RALT1.3 (LED), MX_RALT2.3 (LED), MX_RCTRL1.3 (LED), MX_RCTRL2.3 (LED), MX_RETURN1.3 (LED), MX_RETURN2.3 (LED), MX_RGUI1.3 (LED), MX_RGUI2.3 (LED), MX_RMENU1.3 (LED), MX_RSHIFT1.3 (LED), MX_RSHIFT2.3 (LED), MX_RSHIFT3.3 (LED), MX_RT1.3 (LED), MX_S1.3 (LED), MX_SLOCK1.3 (LED), MX_SP1.3 (LED), MX_SP2.3 (LED), MX_T1.3 (LED), MX_TAB1.3 (LED), MX_U1.3 (LED), MX_UP1.3 (LED), MX_V1.3 (LED), MX_W1.3 (LED), MX_X1.3 (LED), MX_Y1.3 (LED), MX_Z1.3 (LED), MX_[1.3 (LED), MX_\1.3 (LED), MX_\2.3 (LED), MX_]1.3 (LED), MX_`1.3 (LED)
- net CAPS_LEDGND: now also MX_CLOCK3.4 (LEDGND)
- net COL0: now also MX_CLOCK3.2 (ROW), MX_LCTRL3.1 (COL), MX_LGUI3.1 (COL)
- net COL1: now also MX_LALT3.1 (COL)
- net COL3: now also MX_SP3.1 (COL); no longer MX_FN5.1 (COL)
- net COL4: no longer MX_O1.1 (COL)
- net COL5: now also MX_RALT3.1 (COL); no longer MX_/1.1 (COL), MX_RGUI1.1 (COL)
- net COL6: now also MX_RCTRL?.1 (COL), MX_RGUI?.1 (COL); no longer MX_RCTRL1.1 (COL), MX_RMENU1.1 (COL)
- net at D52.2 (A), MX_CLOCK1.2 (ROW), MX_CLOCK2.1 (COL): now also MX_CLOCK3.1 (COL)
- net at D84.2 (A), MX_LCTRL1.2 (ROW), MX_LCTRL2.2 (ROW): now also MX_LCTRL3.2 (ROW)
- net at D85.2 (A), MX_LGUI1.2 (ROW), MX_LGUI2.2 (ROW): now also MX_LGUI3.2 (ROW)
- net at D86.2 (A), MX_LALT1.2 (ROW), MX_LALT2.2 (ROW): now also MX_LALT3.2 (ROW)
- net at D87.2 (A), MX_SP1.2 (ROW), MX_SP2.2 (ROW): now also MX_SP3.2 (ROW)
- net at D91.2 (A), MX_RALT2.2 (ROW), MX_RGUI1.2 (ROW): now also MX_RALT3.2 (ROW)
- net at D81.2 (A), MX_RGUI2.2 (ROW), MX_RMENU1.2 (ROW): now also MX_RGUI?.2 (ROW)
- net at D82.2 (A), MX_RCTRL1.2 (ROW), MX_RCTRL2.2 (ROW): now also MX_RCTRL?.2 (ROW)
- net at MX_PGUP1.2 (ROW): no longer D97.2 (A)
- removed net SLOCK_LEDGND: MX_SLOCK1.4 (LEDGND)
Other:
- moved on the sheet: D1, D10, D100, D101, D108, D11, D111, D112, D113, D12, D13, D14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
