File: proto 8x.kicad_pcb (KiCad board)
At the start: 2 copper layers, 343.7 x 118.3 mm, 122 parts, among them U1 W25Q128JVS, U3 RP2040, Y1 12MHz

Commit message: move f1 + many split layout to complex version, add more board ocmponents
Parts:
- removed MX_BACK2, MX_BACK3, MX_LSHIFT3, MX_NP1, MX_NP3, MX_NP4, MX_NP5, MX_NP6, MX_\2: MX-1U, MX_Alps:MX-1U-NoLED
- removed MX_LALT1, MX_LCTRL1, MX_LGUI1, MX_LSHIFT2, MX_RALT1, MX_RCTRL1, MX_RCTRL3, MX_RGUI1, MX_RMENU1: MX-1.25U, MX_Alps:MX-1.25U-NoLED
- removed MX_SP1: MX-6.25U, MX_Alps:MX-6.25U-NoLED
- added C12: 100nF, Capacitor_SMD:C_0402_1005Metric, B.Cu at (333.4, 107.4)
- added C4: 1uF, Capacitor_SMD:C_0402_1005Metric, B.Cu at (337.8, 113.8)
- added C5: 100nF, Capacitor_SMD:C_0402_1005Metric, B.Cu at (333.4, 105.8)
- added C7: 1uF, Capacitor_SMD:C_0402_1005Metric, B.Cu at (337.8, 114.8)
- added F1: 500mA, Fuse:Fuse_1206_3216Metric, B.Cu at (320.6, 45.2)
- added R5: 27R, Resistor_SMD:R_0603_1608Metric, B.Cu at (333.9, 110.4)
- added R6: 27R, Resistor_SMD:R_0603_1608Metric, B.Cu at (333.9, 112.0)
- added R7: 1k, Resistor_SMD:R_0402_1005Metric, B.Cu at (354.3, 103.8)
- added U2: USBLC6-2SC6, Package_TO_SOT_SMD:SOT-23-6, B.Cu at (326.1, 45.1)
- MX_BACK1: footprint MX_Alps:MX-2U-ReversedStabilizers-NoLED -> MX_Alps:MX-2U-NoLED
- MX_LSHIFT1, MX_RETURN1: footprint MX_Alps:MX-2.25U-ReversedStabilizers-NoLED -> MX_Alps:MX-2.25U-NoLED
- MX_RSHIFT1: footprint MX_Alps:MX-2.75U-ReversedStabilizers-NoLED -> MX_Alps:MX-2.75U-NoLED
- moved Y1 36.4 mm to (358.2, 104.6)
- moved U3 32.8 mm to (345.5, 104.6), turned to -90 degrees
- moved U1 28.5 mm to (335.3, 98.3), turned to -90 degrees
Connections:
- U1 pad 5: (no net) -> SD0
- U1 pad 6: (no net) -> QSPI_CLK
- U1 pad 7: (no net) -> SD3
- U1 pad 8: (no net) -> +3V3
- U3 pad 19: (no net) -> GND
- U3 pad 20: (no net) -> XTAL_IN
- U3 pad 21: (no net) -> XTAL_OUT
- U3 pad 43: +3V3 -> (no net)
- U3 pad 44: +3V3 -> (no net)
- U3 pad 45: +1V1 -> (no net)
- U3 pad 46: D- -> (no net)
- U3 pad 47: D+ -> (no net)
- U3 pad 48: +3V3 -> (no net)
- U3 pad 49: +3V3 -> (no net)
- U3 pad 52: QSPI_CLCK -> QSPI_CLK
- USB1 pad 11: (no net) -> VBUS
- USB1 pad 2: (no net) -> VBUS
- Y1 pad 1: (no net) -> XTAL_0
- Y1 pad 2: (no net) -> GND
- Y1 pad 3: (no net) -> XTAL_IN
- Y1 pad 4: (no net) -> GND
Routing:
- net (no net): track 21.4 -> 0.00 mm
- net CS: track 0.00 -> 18.3 mm
- net VBUS: track 0.00 -> 16.9 mm
- net SD1: track 0.00 -> 16.8 mm
- net XTAL_IN: track 0.00 -> 16.1 mm
- net SD2: track 0.00 -> 15.4 mm
- net SD3: track 0.00 -> 8.84 mm
- net QSPI_CLK: track 0.00 -> 7.41 mm
- net SD0: track 0.00 -> 5.96 mm
- net XTAL_OUT: track 0.00 -> 5.20 mm
- net XTAL_0: track 0.00 -> 2.21 mm
