File: 3u-4.5u-jis/KBD8X-MK2-big-xd.kicad_pcb (KiCad board)
At the start: 2 copper layers, 343.7 x 118.3 mm, 214 parts, among them J1 AVR-ISP-6, Q1 DSS60601MZ4-13, SW1 SW_Push, U1 ATmega32U4-MU, U2 PRTR5V0U2X, Y1 16MHz

Commit message: route part of the right sides, cleanup, add possible jis support lol
Parts:
- added MX_LCTRL1: MX-ALPS-1.5U, MX_Only:MXOnly-1.25U-NoLED, F.Cu at (83.6, 139.7)
- added MX_LCTRL1: MX-ALPS-1.5U, MX_Only:MXOnly-1.25U-NoLED, F.Cu at (50.1, 139.8)
- added MX_LCTRL1: MX-ALPS-1.5U, MX_Only:MXOnly-1.25U-NoLED, F.Cu at (283.4, 139.8)
- added MX_LCTRL1: MX-ALPS-1.5U, MX_Only:MXOnly-1.25U-NoLED, F.Cu at (245.2, 139.8)
- added MX_LCTRL1: MX-ALPS-1.5U, MX_Only:MXOnly-1.25U-NoLED, F.Cu at (269.1, 139.8)
- added MX_LCTRL1: MX-ALPS-1.5U, MX_Only:MXOnly-1.25U-NoLED, F.Cu at (259.5, 139.8)
- added MX_LCTRL1: MX-ALPS-1.5U, MX_Only:MXOnly-1.25U-NoLED, F.Cu at (235.7, 139.8)
- added MX_LCTRL1: MX-ALPS-1.5U, MX_Only:MXOnly-1.75U-NoLED, F.Cu at (54.9, 139.7)
- added MX_LCTRL1: MX-ALPS-1.5U, MX_Only:MXOnly-1.25U-NoLED, F.Cu at (221.4, 139.8)
- added MX_LCTRL1: MX-ALPS-1.5U, MX_Only:MXOnly-1.25U-NoLED, F.Cu at (312.0, 139.8)
- added MX_LCTRL1: MX-ALPS-1.5U, MX_Only:MXOnly-1.25U-NoLED, F.Cu at (107.5, 139.7)
- added MX_LCTRL1: MX-ALPS-1.5U, MX_Only:MXOnly-1.25U-NoLED, F.Cu at (211.7, 139.8)
- added MX_LCTRL1: MX-ALPS-1.5U, MX_Only:MXOnly-1.25U-NoLED, F.Cu at (131.4, 139.8)
- added MX_LCTRL1: MX-ALPS-1.5U, MX_Only:MXOnly-1.25U-NoLED, F.Cu at (93.1, 139.8)
- added MX_LGUI1: MX-ALPS-1U, MX_Only:MXOnly-1U-NoLED, F.Cu at (71.6, 139.8)
- added MX_LGUI1: MX-ALPS-1U, MX_Only:MXOnly-1U-NoLED, F.Cu at (114.6, 139.8)
- added MX_LGUI1: MX-ALPS-1U, MX_Only:MXOnly-1U-NoLED, F.Cu at (290.5, 139.8)
- added MX_RCTRL1: MX-ALPS-1.5U, MX_Only:MXOnly-1.25U-NoLED, F.Cu at (309.7, 139.8)
- added MX_SP2: MX-7U, MX_Alps_Hybrid:MX-3U-ReversedStabilizers-NoLED, F.Cu at (171.8, 139.9)
- renumbered MX_RCTRLe to MX_RCTRL
Routing:
- net ROW10: track 353.9 -> 338.8 mm
- net ROW11: track 335.0 -> 325.1 mm
